File: hardware/BREAD_Slice.kicad_sch (KiCad schematic)
At the start: 15 parts, among them J1 Conn_01x10_Female, J2 I2C_01x04

Commit message: Initial commit
Parts:
- removed J1: Conn_01x10_Female, Connector_PinSocket_2.54mm:PinSocket_1x10_P2.54mm_Horizontal, symbol Connector:Conn_01x10_Female
- removed J2: I2C_01x04, Connector_JST:JST_SH_SM04B-SRSS-TB_1x04-1MP_P1.00mm_Horizontal, symbol SparkFun-Connector:I2C_01x04
- added J1: I2C_01x04, Connector_JST:JST_SH_SM04B-SRSS-TB_1x04-1MP_P1.00mm_Horizontal, symbol SparkFun-Connector:I2C_01x04
- added J2: Conn_01x10_Female, Connector_PinSocket_2.54mm:PinSocket_1x10_P2.54mm_Horizontal, symbol Connector:Conn_01x10_Female
- added J3, J4: Conn_01x02_Socket, symbol Connector:Conn_01x02_Socket
- added Logo1: Logo_Open_Hardware_Small, Symbol:OSHW-Symbol_6.7x6mm_SilkScreen, symbol Graphic:Logo_Open_Hardware_Small
Connections:
- net +12V: now also J2.2 (Pin_2), J2.9 (Pin_9)
- net +5V: now also J1.2 (Pin_2)
- net E_STOP: now also J2.6 (Pin_6)
- net GND: now also J1.1 (Pin_1), J2.1 (Pin_1), J2.10 (Pin_10), J2.5 (Pin_5), J4.2 (Pin_2)
- net I2C_CLK: now also J1.4 (Pin_4), J2.3 (Pin_3)
- net I2C_DAT: now also J1.3 (Pin_3), J2.4 (Pin_4)
- net INT: now also J2.7 (Pin_7)
- net LED: no longer A1.8 (D5)
- net SYNC: now also J2.8 (Pin_8)
- net RESET: now reaches A1.10 (D7)
- net BHI: now reaches A1.13 (D10)
- net BLO: now reaches A1.14 (D11)
- net AHI: now reaches A1.15 (D12)
- net ALO: now reaches A1.16 (D13)
- net FAULT: now reaches A1.9 (D6)
- new net A4947 H-Bridge/OUTA: J3.2 (Pin_2)
- new net A4947 H-Bridge/OUTB: J3.1 (Pin_1)
- new net A4947 H-Bridge/VBB: J4.1 (Pin_1)
- no-connect marks 22 -> 16
Other:
- added sheet A4947 H-Bridge (../A4957_driver.kicad_sch)
