File: hardware/A4957_driver.kicad_sch (KiCad schematic)
At the start: 21 parts, among them Q1 PSMN1R0-30YLC,115, Q2 PSMN1R0-30YLC,115, Q3 PSMN1R0-30YLC,115, Q4 PSMN1R0-30YLC,115, U2 A4957SESTR-T

Commit message: fix(hw): re-point stale library nicknames
These parts exist in KiCad-Master-Lib; the boards referenced libraries that no
longer exist (kml-custom, KML-Custom, and SparkFun libraries that never
contained the part) or names the library has since changed.

KiCad embeds footprint geometry in the .kicad_pcb, so the boards rendered and
fabricated correctly and the rot stayed invisible -- it only surfaces on
update-from-library, or when a generator tries to resolve a nickname.

Nickname/name only. No geometry is changed:

  SparkFun-DiscreteSemi:AP63205 -> KMLib_IC_Power:AP63205WU-7_Buck_Regulator
  SparkFun-LED:WS2812-5050-4PIN -> KMLib_IC_SMD:WS2812-5050-4PIN
  kml-custom:A4957SESTR-T -> KMLib_IC_Power:A4957SESTR-T_Gate_Driver
  kml-custom:QFN-24_ALM -> KMLib_IC_SMD:QFN-24_ALM
  kml-custom:Thermal Pad -> KMLib_Mounting:Thermal_Pad
  kml-custom:WAGO_2606-1104_010-000 -> KMLib_Connectors:2606-1104_010-000_Wago

Only references that failed to resolve were touched. Generic parts (<=4 pins)
and KiCad *-rescue libraries are deliberately excluded: fingerprint matching
cannot distinguish a 2-pin resistor from a 2-pin capacitor, so those are being
done by hand.
Parts:
- U2: footprint kml-custom:QFN-24_ALM -> KMLib_IC_SMD:QFN-24_ALM; symbol kml-custom:A4957SESTR-T -> KMLib_IC_Power:A4957SESTR-T_Gate_Driver
Changed lines of the file:
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@@
 	)
 	(symbol
-		(lib_id "kml-custom:A4957SESTR-T")
+		(lib_id "KMLib_IC_Power:A4957SESTR-T_Gate_Driver")
 		(at 238.76 85.09 0)
 		(mirror y)
@@
 			)
 		)
-		(property "Footprint" "kml-custom:QFN-24_ALM"
+		(property "Footprint" "KMLib_IC_SMD:QFN-24_ALM"
 			(at 238.76 85.09 0)
 			(hide yes)
