File: hardware-4layer/BREAD_Slice.kicad_sch (KiCad schematic)
At the start: 17 parts, among them J1 I2C_01x04, J2 Conn_01x10_Female, J7 2606-1104/010-000, J8 2606-1104/010-000

Commit message: finished initial schematic and board
Parts:
- removed J1: I2C_01x04, Connector_JST:JST_SH_SM04B-SRSS-TB_1x04-1MP_P1.00mm_Horizontal, symbol SparkFun-Connector:I2C_01x04
- removed J8: 2606-1104/010-000, CONN4_2606-1104/010-000_WAG, symbol kml-custom:WAGO_2606-1104_010-000
- added NT1: NetTie_2, NetTie:NetTie-2_SMD_Pad2.0mm, symbol Device:NetTie_2
- C1, C2, C3, C4: footprint Capacitor_SMD:C_1206_3216Metric -> Capacitor_SMD:C_1206_3216Metric_Pad1.33x1.80mm_HandSolder
- D1: PROD_ID (none) -> DIO-12503
- HS1: footprint KML-Custom:Thermal Pad -> kml-custom:Thermal Pad
- J2: renamed from J7; footprint CONN4_2606-1104/010-000_WAG -> kml-custom:CONN4_2606-1104&slash_010-000_WAG
- U1: value ~ -> AP63205
- renumbered J2 to J1
Connections:
- net BHI2 is gone; now on net ALO1: A1.13 (D10)
- net A4947 H-Bridge/OUTA: now also J2.4
- net A4947 H-Bridge/OUTB: now also J2.2
- net ALO1: no longer A1.12 (D9)
- net BHI1: now also A1.12 (D9); no longer A1.9 (D6)
- net BLO1: now also A1.9 (D6); no longer A1.10 (D7)
- net GND: now also J2.1, NT1.1; no longer J1.1 (Pin_1), J1.10 (Pin_10), J1.5 (Pin_5)
- net VBB1: now reaches J2.3
- net AHI1: no longer names the net of A1.11 (D8)
- net AHI2: no longer names the net of A1.15 (D12)
- net ALO2: no longer names the net of A1.16 (D13)
- net BLO2 renamed ALI1
- net E_STOP renamed ESTOP
- net FAULT2: no longer names the net of A1.21 (A2)
- net RESET2: no longer names the net of A1.22 (A3)
- new net GNDPWR: J1.1 (Pin_1), J1.10 (Pin_10), J1.5 (Pin_5), NT1.2
- no-connect marks 10 -> 16
Other:
- removed sheet A4947 H-Bridge1
- sheet A4947 H-Bridge ports: added ALI, GNDA; removed AHI
- note added: "5V Switching Supply"
- note added: "Arduino Nano"
- note added: "Backplane Conn."
- note added: "Color Scheme Legend: ---------------------------------------------------------- color - value - reference ---------------------------------------------------------- • Red - red3 - Analog 5V Supply (e.g., for amps, ADC, references) • Brown - orange1 - Analog Ground (sensor/amp/ADC ground) • Orange - orange3 - Digital 5V Supply (MCU, digital circuits) • Black - black - Digital Ground (MCU ground) •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"
- note added: "Mounting Holes"
- note added: "Pinout Details Arduino Nano: -------------------------------------------------------------------------------------------------------------------- Pin | Function | Limitations/Notes -------------------------------------------------------------------------------------------------------------------- VIN | External Supply Input | External power source 7-12V GND | Ground | First GND pin available for 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"
- note added: "RGB LED"
- moved on the sheet: A1, C1, C2, C3, C4, H1, H2, H3, H4, J2, L1, U1
